File: kiCAD/plantMonitor.kicad_sch (KiCad schematic)
At the start: 10 parts, among them U1 DHT11-1

Commit message: sensors print to json and added trigger debounce
Connections:
- net at U2.3 (SDA): now also A2.13 (SDA/A4); no longer A2.11 (A2)
- net at U2.4 (SCL): now also A2.14 (SCL/A5); no longer A2.10 (A1)

Commit message: added draft diagrams
Parts:
- removed (?) Soil Moisture1: ~, symbol sensorLibrary:Soil_Moisture_Sensor
- removed A2: Arduino_UNO_R2, Module:Arduino_UNO_R2, symbol MCU_Module:Arduino_UNO_R2
- removed LM393-1: ~, symbol sensorLibrary:LM393_Photodiode
- removed R1, R2, R3, R4: 10kΩ, symbol Device:R_Small_US
- removed TEMT1: ~, symbol sensorLibrary:TEMT6000
- removed U1: DHT11-1, Sensor:Aosong_DHT11_5.5x12.0_P2.54mm, symbol Sensor:DHT11
- removed U2: ~, symbol sensorLibrary:LCD1602_I2C
Other:
- added sheet muxSetup (muxSetup.kicad_sch)
- added sheet testSetup (testSetup.kicad_sch)
